File: kicad/linear_rect_driver_panel.kicad_pcb (KiCad board)
At the start: 2 copper layers, 9.5 x 14.8 mm, 11 parts, among them P1 V+, P2 V-, P3 LD+, P4 LD-, Q1 Q_NMOS_GSD, U1 LT3080

Commit message: misc pcb changes
Routing:
- net /Vin: track 30.7 -> 32.6 mm
Other:
- board size 9.5 x 14.8 mm -> 99.9 x 99.9 mm
- board text added: "GitleM. @gmail.com"
- board text added: "GnomeDrive rev. 1.0"
